File: rev_A/esp_prog_uart_autoreset.kicad_pcb (KiCad board)
At the start: 2 copper layers, 30.5 x 25.4 mm, 6 parts, among them J1 UART, J2 ESP, Q1 LMUN2215, Q2 LMUN2215

Commit message: Update to KiCad 6.0
Other:
- net class Default removed
